Commit message: The study of the neck linkage, changed how we should define the robot.

File: src/robbie_description/urdf/robbie.ros2_control.xacro (robot description, xacro)
@@ -7,10 +7,10 @@
 -->
 <robot xmlns:xacro="http://www.ros.org/wiki/xacro">
-  <xacro:macro name="robbie_ros2_control" params="sim headless start_deg">
+  <xacro:macro name="robbie_ros2_control" params="sim headless twist start_deg">
     <ros2_control name="robbie" type="system">
       <hardware>
         <xacro:if value="${sim}">
           <plugin>mujoco_ros2_control/MujocoSystemInterface</plugin>
-          <param name="mujoco_model">$(find robbie_description)/mujoco/scene.xml</param>
+          <param name="mujoco_model">$(find robbie_description)/mujoco/scene_${twist}.xml</param>
           <param name="headless">${headless}</param>
           <param name="sim_speed_factor">1.0</param>

File: src/robbie_description/urdf/robbie.urdf.xacro (robot description, xacro)
@@ -9,4 +9,5 @@
   <xacro:arg name="sim" default="true"/>
   <xacro:arg name="headless" default="false"/>
+  <xacro:arg name="twist" default="ccw"/>   <!-- sim only: the pole, cw or ccw seen from above -->
   <xacro:property name="neck" value="${xacro.load_yaml('$(find robbie_description)/config/neck.yaml')}"/>
   <xacro:property name="pivot_r" value="${neck['sled']['pivot_radius']}"/>
@@ -35,5 +36,5 @@
   <xacro:sled n="3"/>
   <xacro:include filename="$(find robbie_description)/urdf/robbie.ros2_control.xacro"/>
-  <xacro:robbie_ros2_control sim="$(arg sim)" headless="$(arg headless)"
+  <xacro:robbie_ros2_control sim="$(arg sim)" headless="$(arg headless)" twist="$(arg twist)"
                              start_deg="${neck['sled']['start_deg']}"/>
 </robot>
